File: eagle/ArduinoLFO_Main/ArduinoLFO_Main.sch (EAGLE design)
At the start: 23 parts, among them IC1 MCP4922

Commit message: Board Design
Parts:
- removed JP3: OUTB, pinhead:PINHD-1X2
- removed JP4: VREFB, pinhead:PINHD-1X3
- C1: device rcl:CPOL-EUSANYO_C6 -> rcl:CPOL-EUE2.5-7
- R1, R2, R3, R4: device rcl:R-EU_0207/7 -> rcl:R-EU_0204/2V
Connections:
- removed net N$4: IC1.8, U$1.D9
- removed net N$8: IC1.11, JP3.1
- removed net N$9: IC1.10, JP4.1
- net +3V3: no longer JP4.3
- net GND: now also IC1.11; no longer JP3.2, JP4.2
Changed lines of the file:
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@@
 <part name="IC1" library="mylib2" deviceset="MCP4922" device=""/>
 <part name="JP1" library="pinhead" deviceset="PINHD-1X2" device="" value="OUTA"/>
-<part name="JP3" library="pinhead" deviceset="PINHD-1X2" device="" value="OUTB"/>
 <part name="GND1" library="supply1" deviceset="GND" device=""/>
 <part name="GND2" library="supply1" deviceset="GND" device=""/>
 <part name="P+1" library="supply1" deviceset="+5V" device=""/>
 <part name="P+2" library="supply1" deviceset="+5V" device=""/>
-<part name="C1" library="rcl" deviceset="CPOL-EU" device="SANYO_C6" value="100uF"/>
+<part name="C1" library="rcl" deviceset="CPOL-EU" device="E2.5-7" value="100uF"/>
 <part name="GND3" library="supply1" deviceset="GND" device=""/>
-<part name="R1" library="rcl" deviceset="R-EU_" device="0207/7" value="1k"/>
-<part name="R2" library="rcl" deviceset="R-EU_" device="0207/7" value="1k"/>
-<part name="R3" library="rcl" deviceset="R-EU_" device="0207/7" value="1k"/>
-<part name="R4" library="rcl" deviceset="R-EU_" device="0207/7" value="1k"/>
+<part name="R1" library="rcl" deviceset="R-EU_" device="0204/2V" value="1k"/>
+<part name="R2" library="rcl" deviceset="R-EU_" device="0204/2V" value="1k"/>
+<part name="R3" library="rcl" deviceset="R-EU_" device="0204/2V" value="1k"/>
+<part name="R4" library="rcl" deviceset="R-EU_" device="0204/2V" value="1k"/>
 <part name="LED1" library="led" deviceset="LED" device="3MM" value="GREEN"/>
 <part name="LED2" library="led" deviceset="LED" device="3MM" value="GREEN"/>
@@
 <part name="JP9" library="pinhead" deviceset="PINHD-1X3" device="" value="PW"/>
 <part name="P+5" library="supply1" deviceset="+5V" device=""/>
-<part name="JP4" library="pinhead" deviceset="PINHD-1X3" device="" value="VREFB"/>
-<part name="+3V4" library="supply1" deviceset="+3V3" device=""/>
 <part name="FRAME1" library="frames" deviceset="A4L-LOC" device=""/>
 <part name="R5" library="rcl" deviceset="R-EU_" device="0207/7" value="10k"/>
@@
 <instance part="IC1" gate="G$1" x="160.02" y="114.3"/>
 <instance part="JP1" gate="G$1" x="200.66" y="147.32"/>
-<instance part="JP3" gate="G$1" x="200.66" y="114.3"/>
 <instance part="GND1" gate="1" x="180.34" y="88.9"/>
 <instance part="GND2" gate="1" x="190.5" y="88.9"/>
@@
 <instance part="JP9" gate="A" x="43.18" y="93.98" rot="MR0"/>
 <instance part="P+5" gate="1" x="53.34" y="129.54"/>
-<instance part="JP4" gate="A" x="200.66" y="99.06"/>
-<instance part="+3V4" gate="G$1" x="185.42" y="104.14"/>
 <instance part="FRAME1" gate="G$1" x="0" y="0"/>
 <instance part="R5" gate="G$1" x="114.3" y="78.74" rot="R90"/>
@@
 </segment>
 </net>
-<net name="N$4" class="0">
-<segment>
-<pinref part="U$1" gate="G$1" pin="D9"/>
-<wire x1="101.6" y1="106.68" x2="149.86" y2="106.68" width="0.1524" layer="91"/>
-<wire x1="149.86" y1="106.68" x2="149.86" y2="99.06" width="0.1524" layer="91"/>
-<wire x1="149.86" y1="99.06" x2="175.26" y2="99.06" width="0.1524" layer="91"/>
-<wire x1="175.26" y1="99.06" x2="175.26" y2="106.68" width="0.1524" layer="91"/>
-<pinref part="IC1" gate="G$1" pin="8"/>
-<wire x1="175.26" y1="106.68" x2="172.72" y2="106.68" width="0.1524" layer="91"/>
-</segment>
-</net>
 <net name="N$6" class="0">
 <segment>
@@
 </segment>
 </net>
-<net name="N$8" class="0">
-<segment>
-<pinref part="IC1" gate="G$1" pin="11"/>
-<wire x1="172.72" y1="114.3" x2="187.96" y2="114.3" width="0.1524" layer="91"/>
-<wire x1="187.96" y1="114.3" x2="187.96" y2="116.84" width="0.1524" layer="91"/>
-<pinref part="JP3" gate="G$1" pin="1"/>
-<wire x1="187.96" y1="116.84" x2="198.12" y2="116.84" width="0.1524" layer="91"/>
-</segment>
-</net>
-<net name="N$9" class="0">
-<segment>
-<wire x1="187.96" y1="111.76" x2="187.96" y2="101.6" width="0.1524" layer="91"/>
-<wire x1="187.96" y1="101.6" x2="198.12" y2="101.6" width="0.1524" layer="91"/>
-<pinref part="IC1" gate="G$1" pin="10"/>
-<wire x1="172.72" y1="111.76" x2="187.96" y2="111.76" width="0.1524" layer="91"/>
-<pinref part="JP4" gate="A" pin="1"/>
-</segment>
-</net>
 <net name="GND" class="0">
 <segment>
 <pinref part="IC1" gate="G$1" pin="12"/>
 <wire x1="172.72" y1="116.84" x2="180.34" y2="116.84" width="0.1524" layer="91"/>
-<wire x1="180.34" y1="116.84" x2="180.34" y2="91.44" width="0.1524" layer="91"/>
+<wire x1="180.34" y1="116.84" x2="180.34" y2="114.3" width="0.1524" layer="91"/>
 <pinref part="GND1" gate="1" pin="GND"/>
+<pinref part="IC1" gate="G$1" pin="11"/>
+<wire x1="180.34" y1="114.3" x2="180.34" y2="91.44" width="0.1524" layer="91"/>
+<wire x1="172.72" y1="114.3" x2="180.34" y2="114.3" width="0.1524" layer="91"/>
+<junction x="180.34" y="114.3"/>
 </segment>
 <segment>
@@
 <wire x1="198.12" y1="147.32" x2="190.5" y2="147.32" width="0.1524" layer="91"/>
 <wire x1="190.5" y1="147.32" x2="190.5" y2="132.08" width="0.1524" layer="91"/>
-<pinref part="JP3" gate="G$1" pin="2"/>
-<wire x1="190.5" y1="132.08" x2="190.5" y2="114.3" width="0.1524" layer="91"/>
-<wire x1="190.5" y1="114.3" x2="198.12" y2="114.3" width="0.1524" layer="91"/>
-<wire x1="190.5" y1="114.3" x2="190.5" y2="99.06" width="0.1524" layer="91"/>
-<junction x="190.5" y="114.3"/>
-<wire x1="190.5" y1="99.06" x2="198.12" y2="99.06" width="0.1524" layer="91"/>
+<wire x1="190.5" y1="132.08" x2="190.5" y2="91.44" width="0.1524" layer="91"/>
 <pinref part="GND2" gate="1" pin="GND"/>
-<wire x1="190.5" y1="91.44" x2="190.5" y2="99.06" width="0.1524" layer="91"/>
-<junction x="190.5" y="99.06"/>
 <pinref part="JP2" gate="A" pin="2"/>
 <wire x1="198.12" y1="132.08" x2="190.5" y2="132.08" width="0.1524" layer="91"/>
 <junction x="190.5" y="132.08"/>
-<pinref part="JP4" gate="A" pin="2"/>
 </segment>
 <segment>
@@
 <wire x1="182.88" y1="58.42" x2="182.88" y2="68.58" width="0.1524" layer="91"/>
 </segment>
-<segment>
-<pinref part="JP4" gate="A" pin="3"/>
-<wire x1="198.12" y1="96.52" x2="185.42" y2="96.52" width="0.1524" layer="91"/>
-<pinref part="+3V4" gate="G$1" pin="+3V3"/>
-<wire x1="185.42" y1="96.52" x2="185.42" y2="101.6" width="0.1524" layer="91"/>
-</segment>
-</net>
+</net>

Commit message: Main Boardはんだ付け完了
Parts:
- removed JP10: PWR_OUT, pinhead:PINHD-1X3
- added C2: 0.1uF, rcl:C-EU025-024X044
- added PO: PWR_OUT, con-amp-quick:MA03S
- JP1, JP5: device pinhead:PINHD-1X2 -> my_pinhead:PINHD-1X2
- JP2: device pinhead:PINHD-1X3 -> my_pinhead:PINHD-1X3
- JP6: value WaveShape -> WavShpe; device pinhead:PINHD-1X2 -> my_pinhead:PINHD-1X2
- JP7: device pinhead:PINHD-1X2 -> con-amp-quick:MA02
- LED1: value GREEN -> LED1
- LED2: value GREEN -> LED2
- LED3: value GREEN -> LED3
- LED4: value GREEN -> LED4
Connections:
- removed net N$5: JP8.2, U$1.A0
- new net N$4: JP8.3, U$1.A0
- net +3V3: now also PO-2.S; no longer JP10.2
- net +5V: now also C2.1, JP9.2, PO-1.S; no longer JP10.1, JP9.1
- net GND: now also C2.2, IC1.8, JP8.2, PO-3.S; no longer JP10.3, JP8.3
- net N$10: now also JP9.1; no longer JP9.2
Other:
- moved on the sheet: C1, JP7
