File: eagle/ArduinoLFO_Output_Board/ArduinoLFO_Output_Board.brd (EAGLE design)
At the start: 70.8 x 45.7 mm, 29 parts, among them IC1 NJU7032, IC2 NJU7032

Commit message: はんだ付け完了
Routing:
- net N$8: track 35.6 -> 32.6 mm
Changed lines of the file:
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@@
 <wire x1="27.94" y1="15.24" x2="27.94" y2="17.78" width="0.4064" layer="16"/>
 <wire x1="27.94" y1="17.78" x2="35.56" y2="17.78" width="0.4064" layer="16"/>
-<wire x1="33.02" y1="27.94" x2="27.94" y2="27.94" width="0.4064" layer="16"/>
-<wire x1="27.94" y1="27.94" x2="27.94" y2="17.78" width="0.4064" layer="16"/>
 <wire x1="27.94" y1="15.24" x2="27.94" y2="7.62" width="0.4064" layer="16"/>
+<wire x1="27.94" y1="17.78" x2="27.94" y2="22.86" width="0.4064" layer="16"/>
+<wire x1="27.94" y1="22.86" x2="33.02" y2="27.94" width="0.4064" layer="16"/>
 </signal>
 <signal name="N$9">
